File: Custom_PCB/custom-pcb.kicad_pcb (KiCad board)
At the start: 2 copper layers, 33.9 x 82.4 mm, 26 parts, among them Q1 IRLML0100

Commit message: PCB
Other:
- board text added: "Jorge De Los Santos Razo 09/15/2025"
- board text removed: "Jorge De Los Santos Razo 09/09/2025"
Changed lines of the file:
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@@
 		(layer "Edge.Cuts")
 	)
-	(gr_text "Jorge De Los Santos Razo\n09/09/2025"
+	(gr_text "Jorge De Los Santos Razo\n09/15/2025"
 		(at 141 118.5 90)
 		(layer "F.SilkS")

Commit message: removed fiducials
Parts:
- removed FID1, FID2, FID3: FIDUCIAL_1MM, Adafruit eInk Breakout Friend:FIDUCIAL_1MM

Commit message: added a footprint
Parts:
- EINK1: footprint Adafruit eInk Breakout Friend:EINK_24PIN -> Adafruit eInk Breakout Friend:FPC-SMD_P0.50-24P_XJ-FGS
- moved EINK1 0.87 mm to (127.8, 58.6)
