File: Custom_PCB/custom-pcb.kicad_sch (KiCad schematic)
At the start: 26 parts, among them Q1 IRLML0100

Commit message: removed fiducials
Parts:
- removed FID1, FID2, FID3: FIDUCIAL_1MM, Adafruit eInk Breakout Friend:FIDUCIAL_1MM, symbol Adafruit eInk Breakout Friend-eagle-import:FIDUCIAL_1MM
Changed lines of the file:
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@@
-	)
-	(symbol
-		(lib_id "Adafruit eInk Breakout Friend-eagle-import:FIDUCIAL_1MM")
-		(at 132.08 189.23 0)
-		(unit 1)
-		(exclude_from_sim no)
-		(in_bom yes)
-		(on_board yes)
-		(dnp no)
-		(property "Reference" "FID1"
-			(at 132.08 189.23 0)
-			(effects
-				(font
-					(size 1.27 1.27)
-				)
-				(hide yes)
-			)
-		)
-		(property "Value" "FIDUCIAL_1MM"
-			(at 132.08 189.23 0)
-			(effects
-				(font
-					(size 1.27 1.27)
-				)
-				(hide yes)
-			)
-		)
-		(property "Footprint" "Adafruit eInk Breakout Friend:FIDUCIAL_1MM"
-			(at 132.08 189.23 0)
-			(effects
-				(font
-					(size 1.27 1.27)
-				)
-				(hide yes)
-			)
-		)
-		(property "Datasheet" ""
-			(at 132.08 189.23 0)
-			(effects
-				(font
-					(size 1.27 1.27)
-				)
-				(hide yes)
-			)
-		)
-		(property "Description" ""
-			(at 132.08 189.23 0)
-			(effects
-				(font
-					(size 1.27 1.27)
-				)
-				(hide yes)
-			)
-		)
-		(instances
-			(project "custo-pcb"
-				(path "/899d7992-9a04-47c7-8d18-5535e976d813"
-					(reference "FID1")
-					(unit 1)
-				)
-			)
-		)
 	)
 	(symbol
@@
 	)
 	(symbol
-		(lib_id "Adafruit eInk Breakout Friend-eagle-import:FIDUCIAL_1MM")
-		(at 148.59 189.23 0)
-		(unit 1)
-		(exclude_from_sim no)
-		(in_bom yes)
-		(on_board yes)
-		(dnp no)
-		(property "Reference" "FID3"
-			(at 148.59 189.23 0)
-			(effects
-				(font
-					(size 1.27 1.27)
-				)
-				(hide yes)
-			)
-		)
-		(property "Value" "FIDUCIAL_1MM"
-			(at 148.59 189.23 0)
-			(effects
-				(font
-					(size 1.27 1.27)
-				)
-				(hide yes)
-			)
-		)
-		(property "Footprint" "Adafruit eInk Breakout Friend:FIDUCIAL_1MM"
-			(at 148.59 189.23 0)
-			(effects
-				(font
-					(size 1.27 1.27)
-				)
-				(hide yes)
-			)
-		)
-		(property "Datasheet" ""
-			(at 148.59 189.23 0)
-			(effects
-				(font
-					(size 1.27 1.27)
-				)
-				(hide yes)
-			)
-		)
-		(property "Description" ""
-			(at 148.59 189.23 0)
-			(effects
-				(font
-					(size 1.27 1.27)
-				)
-				(hide yes)
-			)
-		)
-		(instances
-			(project "custo-pcb"
-				(path "/899d7992-9a04-47c7-8d18-5535e976d813"
-					(reference "FID3")
-					(unit 1)
-				)
-			)
-		)
-	)
-	(symbol
 		(lib_id "power:GND")
 		(at 163.83 113.03 0)
@@
 					(unit 1)
 				)
-			)
-		)
-	)
-	(symbol
-		(lib_id "Adafruit eInk Breakout Friend-eagle-import:FIDUCIAL_1MM")
-		(at 142.24 189.23 0)
-		(unit 1)
-		(exclude_from_sim no)
-		(in_bom yes)
-		(on_board yes)
-		(dnp no)
-		(property "Reference" "FID2"
-			(at 142.24 189.23 0)
-			(effects
-				(font
-					(size 1.27 1.27)
-				)
-				(hide yes)
-			)
-		)
-		(property "Value" "FIDUCIAL_1MM"
-			(at 142.24 189.23 0)
-			(effects
-				(font
-					(size 1.27 1.27)
-				)
-				(hide yes)
-			)
-		)
-		(property "Footprint" "Adafruit eInk Breakout Friend:FIDUCIAL_1MM"
-			(at 142.24 189.23 0)
-			(effects
-				(font
-					(size 1.27 1.27)
-				)
-				(hide yes)
-			)
-		)
-		(property "Datasheet" ""
-			(at 142.24 189.23 0)
-			(effects
-				(font
-					(size 1.27 1.27)
-				)
-				(hide yes)
-			)
-		)
-		(property "Description" ""
-			(at 142.24 189.23 0)
-			(effects
-				(font
-					(size 1.27 1.27)
-				)
-				(hide yes)
-			)
-		)
-		(instances
-			(project "custo-pcb"
-				(path "/899d7992-9a04-47c7-8d18-5535e976d813"
-					(reference "FID2")
-					(unit 1)
-				)

Commit message: small change to schematic
Parts:
- EINK1: footprint Adafruit eInk Breakout Friend:EINK_24PIN -> Adafruit eInk Breakout Friend:FPC-SMD_P0.50-24P_XJ-FGS
Changed lines of the file:
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@@
 			)
 		)
-		(property "Footprint" "Adafruit eInk Breakout Friend:EINK_24PIN"
+		(property "Footprint" "Adafruit eInk Breakout Friend:FPC-SMD_P0.50-24P_XJ-FGS"
 			(at 207.01 143.51 0)
 			(effects
